File: Sharp_DistanceSensor/ECAD/MCU_StepperDriverPCB/MCU_StepperDriverPCB.kicad_pcb (KiCad board)
At the start: 2 copper layers, 62.5 x 57.5 mm, 26 parts, among them J1 Conn_01x02, J2 Conn_01x02_Female, J3 Conn_01x02_Female, J4 Conn_01x05_Female, U1 TA78L05F, U2 STM32_BluePill_PortView

Commit message: MCAD: Added missing parts of sensor assembly. ECAD: updated PCB for MCU and stepper motor driver. SW: Implemented functionality to perform 360deg scans.
Parts:
- A1: value Pololu_Breakout_A4988 -> Watterott SilentStepStick TMC2100
- U2: moved to B.Cu
- moved C5 15.4 mm to (126.6, 107.8), turned to 0 degrees
- moved C6 9.21 mm to (134.9, 113.7), turned to 270 degrees
- moved D12 8.29 mm to (134.9, 109.1)
- moved D1 4.26 mm to (164.4, 97.5)
- moved U1 4.06 mm to (164.4, 102.8), turned to 90 degrees
Connections:
- net /STD_Dir renamed /STMD_Dir
- net /STD_En renamed /STMD_En
- net /STD_Step renamed /STMD_Step
- U1 pad 1: Net-(C2-Pad1) -> +5V
- U1 pad 3: +5V -> Net-(C2-Pad1)
- U2 pad 38: /Light_Barrier -> Net-(C6-Pad1)
- U2 pad 39: Net-(C6-Pad1) -> GND
Routing:
- net /AN_Distance: track 17.5 -> 36.6 mm
- net /Light_Barrier: track 39.9 -> 21.1 mm, vias 0 -> 2
- net /STMD_Step: track 27.5 -> 9.49 mm
- net /STMD_Dir: track 26.3 -> 10.0 mm
- net GND: track 11.6 -> 27.5 mm
- net /STMD_En: track 25.1 -> 10.5 mm
- net Net-(D7-Pad2): track 25.2 -> 10.8 mm
- net +5V: track 90.8 -> 85.6 mm
- net Net-(C2-Pad1): track 13.9 -> 18.5 mm
